File: FN32ROV-XEBook-KiCad.kicad_pcb (KiCad board)
At the start: 2 copper layers, 66 x 56 mm, 64 parts, among them J2 USB-C 16P, Q1 UMH3NTN, Q2 DMP2035U-7, Q3 DMG2302U, U1 ESP32-WROVER-IE-N16R8, U2 CP2102N-A02-GQFN24R, U3 74LS07DR, U4 74LS07DR, U5 XC6220B331MR

Commit message: Normalize 10k/10K resistor value casing, add fab output for JLCPCB assembly order
- Normalize R1-R3/R6/R12/R22 Value from "10k" to "10K" so the BOM groups
  correctly with the other 10K resistors instead of splitting into two lines
- Add Fab/ with Gerbers, PTH/NPTH drill files, pick-and-place, and BOM
  (grouped + JLCPCB-ready with LCSC part numbers) for the v1.0 assembly order
Parts:
- R1, R12, R2, R22, R3, R6: value 10k -> 10K
Changed lines of the file:
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@@
 			)
 		)
-		(property "Value" "10k"
+		(property "Value" "10K"
 			(at 0 1.17 0)
 			(layer "F.Fab")
@@
 			)
 		)
-		(property "Value" "10k"
+		(property "Value" "10K"
 			(at 0 1.17 0)
 			(layer "F.Fab")
@@
 			)
 		)
-		(property "Value" "10k"
+		(property "Value" "10K"
 			(at 0 1.17 0)
 			(layer "F.Fab")
@@
 			)
 		)
-		(property "Value" "10k"
+		(property "Value" "10K"
 			(at 0 1.17 0)
 			(layer "F.Fab")
@@
 			)
 		)
-		(property "Value" "10k"
+		(property "Value" "10K"
 			(at 0 1.17 0)
 			(layer "F.Fab")
@@
 			)
 		)
-		(property "Value" "10k"
+		(property "Value" "10K"
 			(at 0 1.17 90)
 			(layer "F.Fab")
