File: FN32ROV-XEBook-KiCad.kicad_pcb (KiCad board)
At the start: 2 copper layers, 66 x 56 mm, 64 parts, among them J2 USB-C 16P, Q1 UMH3NTN, Q2 DMP2035U-7, Q3 DMG2302U, U1 ESP32-WROVER-E-N16R8, U2 CP2102N-A02-GQFN24R, U3 74LS07DR, U4 74LS07DR, U5 XC6220B331MR

Commit message: Add TP1 SIO audio take-off pad for PokeyMax and re-export fab
A 2.0mm through-hole pad (1.0mm drill) on SIO_AUDIN at (80.475, 56.475),
routed back to J_SIO1 pad 10, so the PokeyMax J2 pin 4 wire has a proper
solder point instead of being tacked onto the back of the IDC header.

Sits in the open area right of J_SIO1, centred in a GND stitching-via cell
above the USB-C connector: 0.82mm to the four nearest vias, 1.1mm clear of
each via column along the route. Silkscreens SIO_AUDIN; the reference is
set not to print.

Marked exclude-from-BOM and exclude-from-position-files, so the BOM stays
at 30 rows and the pick-and-place at 60 placements -- both byte-identical
to the previous 1.1 export, and the hand-mapped PCBWay BOM needs no
revision.

Verification: netlist has TP1 pin 1 on /SIO_AUDIN alongside C3 pin 1 and
J_SIO1 pad 10; DRC reports 0 unconnected, 0 schematic-parity and no
violations involving TP1; no existing pad changed position or net
(280 -> 281 pads, the addition is TP1). Zones refilled, which also cleared
10 pre-existing stale-fill violations (4 hole-clearance, 4 starved-thermal,
2 footprint issues) -- total DRC went 22 -> 12, the remainder all
pre-existing and unrelated.

Fab re-exported into Gerbers-FN32ROV-XEBook-1.1 with the documented
settings (--subtract-soldermask, %LPC=1 confirmed). Against the previous
export only F.Cu, B.Cu, F/B mask, F/B silkscreen and the PTH drill differ;
Edge.Cuts, both paste layers, the NPTH drill and the job file are
unchanged. The PTH drill gains exactly one hole.

Co-Authored-By: Claude Opus 5 (1M context) <noreply@anthropic.com>
Parts:
- added TP1: SIO_AUDIN, TestPoint:TestPoint_THTPad_D2.0mm_Drill1.0mm, F.Cu at (80.5, 56.5)
Routing:
- net /SIO_AUDIN: track 14.4 -> 27.9 mm
Changed lines of the file:
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@@
 		)
 	)
+	(footprint "TestPoint:TestPoint_THTPad_D2.0mm_Drill1.0mm"
+		(layer "F.Cu")
+		(at 80.475 56.475)
+		(descr "THT pad as test Point, diameter 2.0mm, hole diameter 1.0mm")
+		(tags "test point THT pad")
+		(property "Reference" "TP1"
+			(at 0 2.6 0)
+			(layer "F.SilkS")
+			(hide yes)
+			(effects
+				(font
+					(size 1 1)
+					(thickness 0.15)
+				)
+			)
+		)
+		(property "Value" "SIO_AUDIN"
+			(at 0 2.525 0)
+			(layer "F.SilkS")
+			(effects
+				(font
+					(size 0.8 0.8)
+					(thickness 0.13)
+				)
+			)
+		)
+		(property "Datasheet" ""
+			(at 0 0 0)
+			(unlocked yes)
+			(layer "F.Fab")
+			(hide yes)
+			(effects
+				(font
+					(size 1.27 1.27)
+					(thickness 0.15)
+				)
+			)
+		)
+		(property "Description" "test point"
+			(at 0 0 0)
+			(unlocked yes)
+			(layer "F.Fab")
+			(hide yes)
+			(effects
+				(font
+					(size 1.27 1.27)
+					(thickness 0.15)
+				)
+			)
+		)
+		(attr exclude_from_pos_files exclude_from_bom)
+		(fp_circle
+			(center 0 0)
+			(end 0 1.2)
+			(stroke
+				(width 0.12)
+				(type solid)
+			)
+			(fill no)
+			(layer "F.SilkS")
+		)
+		(fp_circle
+			(center 0 0)
+			(end 1.5 0)
+			(stroke
+				(width 0.05)
+				(type solid)
+			)
+			(fill no)
+			(layer "F.CrtYd")
+		)
+		(fp_text user "${REFERENCE}"
+			(at 0 -2 0)
+			(layer "F.Fab")
+			(effects
+				(font
+					(size 1 1)
+					(thickness 0.15)
+				)
+			)
+		)
+		(pad "1" thru_hole circle
+			(at 0 0)
+			(size 2 2)
+			(drill 1)
+			(layers "*.Cu" "*.Mask")
+			(remove_unused_layers no)
+			(net 4 "/SIO_AUDIN")
+			(pinfunction "1")
+			(pintype "passive")
+		)
+		(embedded_fonts no)
+	)
 	(footprint "Capacitor_SMD:C_0402_1005Metric"
 		(layer "F.Cu")
@@
 	)
 	(segment
+		(start 80.475 48.46)
+		(end 80.475 56.475)
+		(width 0.2)
+		(layer "F.Cu")
+		(net 4)
+	)
+	(segment
 		(start 74.1425 44.5016)
 		(end 74.1425 46.19)
@@
 	)
 	(segment
+		(start 75.4125 47.46)
+		(end 79.475 47.46)
+		(width 0.2)
+		(layer "F.Cu")
+		(net 4)
+	)
+	(segment
 		(start 72.3878 43.7099)
 		(end 73.3508 43.7099)
 		(width 0.2)
 		(layer "F.Cu")
+		(net 4)
+	)
+	(segment
+		(start 79.475 47.46)
+		(end 80.475 48.46)
+		(width 0.2)
+		(layer "F.Cu")

Commit message: Silkscreen: add pin-1 markers to the cable headers
Marks pin 1 on J_BTN1, J_LED1 and J_SD1 so the three daughter-board
cables cannot be seated backwards during assembly.

Verified against the previous commit: footprints, pads, copper segments,
vias and zone definitions are all unchanged. Only F.SilkS text was added
(plus zone refills and uuid churn from the save).

Co-Authored-By: Claude Opus 5 (1M context) <noreply@anthropic.com>
Other:
- board text added: "1"
Changed lines of the file:
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@@
 		(tags "connector JST PH horizontal")
 		(property "Reference" "J_BTN1"
-			(at 3 -2.55 0)
+			(at 5.5 -2.55 0)
 			(layer "F.SilkS")
 			(effects
@@
 		(tags "connector JST PH horizontal")
 		(property "Reference" "J_LED1"
-			(at 3 -2.55 0)
+			(at 6 -2.55 0)
 			(layer "F.SilkS")
 			(effects
@@
 		(layer "Edge.Cuts")
 	)
+	(gr_text "1"
+		(at 60 71 0)
+		(layer "F.SilkS")
+		(effects
+			(font
+				(size 1 1)
+				(thickness 0.15)
+			)
+		)
+	)
+	(gr_text "1"
+		(at 47.5 71 0)
+		(layer "F.SilkS")
+		(effects
+			(font
+				(size 1 1)
+				(thickness 0.15)
+			)
+		)
+	)
+	(gr_text "1"
+		(at 29 34 270)
+		(layer "F.SilkS")
+		(effects
+			(font
+				(size 1 1)
+				(thickness 0.15)
+			)
+		)
+	)
 	(segment
