File: FN32ROV-XEBook-KiCad.kicad_sch (KiCad schematic)
At the start: 60 parts, among them J2 USB-C 16P, Q1 UMH3NTN, Q2 DMP2035U-7, Q3 DMG2302U, U1 ESP32-WROVER-IE-N16R8, U2 CP2102N-A02-GQFN24R, U3 74LS07DR, U4 74LS07DR, U5 XC6220B331MR

Commit message: Resize R13 to 2.7k for the LED boards green WiFi LED, document the LED board interface
The WiFi status LED moved to the new FN32ROV-XEBook-LED-KiCad daughter board and
changed color from white to green, which has a lower forward voltage (~2.2V vs
~2.9V). R13 needed to grow from 1k to 2.7k to keep the current in the same range
as the original design. Also documents the sibling LED board repo and the
per-channel resistor rationale in CLAUDE.md.

Co-Authored-By: Claude Sonnet 5 <noreply@anthropic.com>
Claude-Session: https://claude.ai/code/session_011E5FphyrLWBpYvbXpCPZfr
Parts:
- R13: value 1k -> 2.7k
Changed lines of the file:
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@@
 			)
 		)
-		(property "Value" "1k"
+		(property "Value" "2.7k"
 			(at 50.8 294.64 90)
 			(effects

Commit message: Replace D7/D8 diode part to fix SOD-323/SOD-123W package mismatch
PCBWay's assembly review caught that PMEG2010ER,115 (the part specified
for D7/D8) is only manufactured in SOD-123W, not the SOD-323 footprint
used on this board. Rather than swap the PCB footprint (which would
require re-routing around a nearby USB_D+ trace and re-exporting
gerbers), swapped the part instead: Nexperia PMEG2010BEA,115
(LCSC C455041) is a direct electrical equivalent (20V/1A Schottky, low
Vf) genuinely packaged in SOD-323, matching the existing footprint.
Board layout and gerbers are unaffected (value text lives on F.Fab).

Also includes the filled-in Customer Reply column for PCBWay's BOM
quote questions (this diode fix, three benign capacitor voltage-rating
upgrades, sourcing for J_SIO1, and flagging that their R13 quote used a
stale pre-2.7k BOM revision).

Co-Authored-By: Claude Sonnet 5 <noreply@anthropic.com>
Claude-Session: https://claude.ai/code/session_01GM9FQ1pLMMKCV3Qfiq1ore
Parts:
- D7, D8: value PMEG2010ER,115 -> PMEG2010BEA,115
Changed lines of the file:
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@@
 			)
 		)
-		(property "Value" "PMEG2010ER,115"
+		(property "Value" "PMEG2010BEA,115"
 			(at 153.67 335.28 0)
 			(effects
@@
 			)
 		)
-		(property "Value" "PMEG2010ER,115"
+		(property "Value" "PMEG2010BEA,115"
 			(at 153.924 307.34 0)
 			(effects
